File: pinboard.kicad_pcb (KiCad board)
At the start: 2 copper layers, 263.4 x 109.4 mm, 27 parts, among them SW1 SW_Choc_1u, SW10 SW_Choc_1u, SW11 SW_Choc_1u, SW12 SW_Choc_1u, SW13 SW_Choc_1u, SW14 SW_Choc_1u, SW15 SW_Choc_1u, SW16 SW_Choc_1u, SW17 SW_Choc_1u, SW18 SW_Choc_1u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

Commit message: v1.1
Parts:
- SW1, SW10, SW11, SW12, SW13, SW14, SW15, SW16, SW17, SW18, SW19, SW2, SW20, SW21, SW22, SW23, SW24, SW3, SW4, SW5, SW6, SW7, SW8, SW9: footprint rznkbd-switches:SW_Choc_v1v2_1u_Hotswap_NonReversible -> rznkbd-switches:SW_Choc_v1v2_1u_Solder_Hotswap
- moved SW22 0.64 mm to (206.8, 141.3)
- moved SW2 0.64 mm to (77.7, 143.2)
- moved SW23 0.64 mm to (230.7, 178.6)
- moved SW5 0.64 mm to (102.8, 119.2)
- moved SW18 0.64 mm to (242.7, 136.1)
- moved SW20 0.64 mm to (226.4, 144.9)
- moved SW24 0.64 mm to (213.4, 183.3)
- moved SW8 0.64 mm to (133.2, 144.9)
- moved SW3 0.64 mm to (82.1, 126.8)
- moved SW12 0.64 mm to (145.9, 184.4)
- moved SW14 0.64 mm to (281.8, 143.2)
- moved SW21 0.64 mm to (222.0, 128.5)
- moved SW9 0.64 mm to (137.6, 128.5)
- moved U1 0.64 mm to (179.8, 136.4)
- moved SW7 0.64 mm to (121.3, 119.7)
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Connections:
- SW1 pad 1: sw1 -> gnd
- SW1 pad 2: gnd -> sw1
- SW10 pad 1: sw10 -> gnd
- SW10 pad 2: gnd -> sw10
- SW11 pad 1: sw11 -> gnd
- SW11 pad 2: gnd -> sw11
- SW12 pad 1: sw12 -> gnd
- SW12 pad 2: gnd -> sw12
- SW13 pad 1: sw13 -> gnd
- SW13 pad 2: gnd -> sw13
- SW14 pad 1: sw14 -> gnd
- SW14 pad 2: gnd -> sw14
- SW15 pad 1: sw15 -> gnd
- SW15 pad 2: gnd -> sw15
- SW16 pad 1: sw16 -> gnd
- SW16 pad 2: gnd -> sw16
- SW17 pad 1: sw17 -> gnd
- SW17 pad 2: gnd -> sw17
- SW18 pad 1: sw18 -> gnd
- SW18 pad 2: gnd -> sw18
- SW19 pad 1: sw19 -> gnd
- SW19 pad 2: gnd -> sw19
- SW2 pad 1: sw2 -> gnd
- SW2 pad 2: gnd -> sw2
- SW20 pad 1: sw20 -> gnd
- SW20 pad 2: gnd -> sw20
- SW21 pad 1: sw21 -> gnd
- SW21 pad 2: gnd -> sw21
- SW22 pad 1: sw22 -> gnd
- SW22 pad 2: gnd -> sw22
- SW23 pad 1: sw23 -> gnd
- SW23 pad 2: gnd -> sw23
- SW24 pad 1: sw24 -> gnd
- SW24 pad 2: gnd -> sw24
- SW3 pad 1: sw3 -> gnd
- SW3 pad 2: gnd -> sw3
- SW4 pad 1: sw4 -> gnd
- SW4 pad 2: gnd -> sw4
- SW5 pad 1: sw5 -> gnd
- SW5 pad 2: gnd -> sw5
- SW6 pad 1: sw6 -> gnd
- SW6 pad 2: gnd -> sw6
- SW7 pad 1: sw7 -> gnd
- SW7 pad 2: gnd -> sw7
- SW8 pad 1: sw8 -> gnd
- SW8 pad 2: gnd -> sw8
- SW9 pad 1: sw9 -> gnd
- SW9 pad 2: gnd -> sw9
Routing:
- net sw13: track 120.6 -> 138.8 mm
- net sw15: track 118.9 -> 136.1 mm
- net sw6: track 75.7 -> 92.9 mm
- net sw3: track 114.7 -> 131.9 mm
- net sw5: track 111.1 -> 128.3 mm
- net sw1: track 122.9 -> 140.1 mm
- net sw4: track 96.0 -> 113.1 mm
- net sw20: track 75.1 -> 92.2 mm
- net sw10: track 13.9 -> 31.0 mm
- net sw8: track 60.9 -> 78.0 mm
- net sw19: track 116.1 -> 133.2 mm
- net sw22: track 33.3 -> 50.2 mm
- net sw18: track 100.8 -> 117.7 mm
- net sw7: track 91.3 -> 108.2 mm
- net sw17: track 122.7 -> 139.6 mm
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- added copper zone on B.Cu, net gnd
Other:
- board text added: "pinboard v1.1 by razen made for pinchord layout"
- board text removed: "pinboard v1.0 by razen made for pinchord layout"
