File: pinboard.kicad_sch (KiCad schematic)
At the start: 25 parts, among them SW1 SW_Choc_1u, SW10 SW_Choc_1u, SW11 SW_Choc_1u, SW12 SW_Choc_1u, SW13 SW_Choc_1u, SW14 SW_Choc_1u, SW15 SW_Choc_1u, SW16 SW_Choc_1u, SW17 SW_Choc_1u, SW18 SW_Choc_1u, SW19 SW_Choc_1u, SW2 SW_Choc_1u, SW20 SW_Choc_1u, SW21 SW_Choc_1u, SW22 SW_Choc_1u, SW23 SW_Choc_1u, SW24 SW_Choc_1u, SW3 SW_Choc_1u, SW4 SW_Choc_1u, SW5 SW_Choc_1u, SW6 SW_Choc_1u, SW7 SW_Choc_1u, SW8 SW_Choc_1u, SW9 SW_Choc_1u, U1 RP2040-Zero

Commit message: v1.1
Parts:
- SW1, SW10, SW11, SW12, SW13, SW14, SW15, SW16, SW17, SW18, SW19, SW2, SW20, SW21, SW22, SW23, SW24, SW3, SW4, SW5, SW6, SW7, SW8, SW9: footprint rznkbd-switches:SW_Choc_v1v2_1u_Hotswap_NonReversible -> rznkbd-switches:SW_Choc_v1v2_1u_Solder_Hotswap
Connections:
- net gnd: now also SW1.1, SW10.1, SW11.1, SW12.1, SW13.1, SW14.1, SW15.1, SW16.1, SW17.1, SW18.1, SW19.1, SW2.1, SW20.1, SW21.1, SW22.1, SW23.1, SW24.1, SW3.1, SW4.1, SW5.1, SW6.1, SW7.1, SW8.1, SW9.1; no longer SW1.2, SW10.2, SW11.2, SW12.2, SW13.2, SW14.2, SW15.2, SW16.2, SW17.2, SW18.2, SW19.2, SW2.2, SW20.2, SW21.2, SW22.2, SW23.2, SW24.2, SW3.2, SW4.2, SW5.2, SW6.2, SW7.2, SW8.2, SW9.2
- net sw1: now also SW1.2; no longer SW1.1
- net sw10: now also SW10.2; no longer SW10.1
- net sw11: now also SW11.2; no longer SW11.1
- net sw12: now also SW12.2; no longer SW12.1
- net sw13: now also SW13.2; no longer SW13.1
- net sw14: now also SW14.2; no longer SW14.1
- net sw15: now also SW15.2; no longer SW15.1
- net sw16: now also SW16.2; no longer SW16.1
- net sw17: now also SW17.2; no longer SW17.1
- net sw18: now also SW18.2; no longer SW18.1
- net sw19: now also SW19.2; no longer SW19.1
- net sw2: now also SW2.2; no longer SW2.1
- net sw20: now also SW20.2; no longer SW20.1
- net sw21: now also SW21.2; no longer SW21.1
- net sw22: now also SW22.2; no longer SW22.1
- net sw23: now also SW23.2; no longer SW23.1
- net sw24: now also SW24.2; no longer SW24.1
- net sw3: now also SW3.2; no longer SW3.1
- net sw4: now also SW4.2; no longer SW4.1
- net sw5: now also SW5.2; no longer SW5.1
- net sw6: now also SW6.2; no longer SW6.1
- net sw7: now also SW7.2; no longer SW7.1
- net sw8: now also SW8.2; no longer SW8.1
- net sw9: now also SW9.2; no longer SW9.1
